Commit message: Rebase from 'upstream'

File: mir_description/urdf/include/common.gazebo.xacro (robot description, xacro)
@@ -5,5 +5,5 @@
       <plugin name="gazebo_ros_control" filename="libgazebo_ros_control.so">
         <xacro:unless value="${robot_namespace == ''}">
-          <robotNamespace>($robot_namespace)</robotNamespace>
+          <robotNamespace>${robot_namespace}</robotNamespace>
         </xacro:unless>
         <controlPeriod>0.001</controlPeriod>

File: mir_description/urdf/include/mir_100_v1.urdf.xacro (robot description, xacro)
@@ -1,4 +1,15 @@
 <?xml version="1.0"?>
 <robot xmlns:xacro="http://ros.org/wiki/xacro">
+  <!-- The gazebo_ros_laser plugin does the following:
+       - If the ROS parameter 'tf_prefix' is set, it prepends the
+       - tf_prefix in front of the frameName.
+       - Otherwise, it prepends the robotNamespace.
+       The robotNamespace gets automatically set if you start the
+       spawn_model node inside a namespace. In this case, set
+       prepend_prefix_to_laser_frame to 'false', otherwise the
+       resulting frameName will have two prefixes prepended.
+       If you don't start spawn_model inside a namespace but have a
+       non-empty prefix, set prepend_prefix_to_laser_frame to 'true'. -->
+  <xacro:arg name="prepend_prefix_to_laser_frame" default="false" />
   <xacro:include filename="$(find mir_description)/urdf/include/common_properties.urdf.xacro" />
   <xacro:include filename="$(find mir_description)/urdf/include/imu.gazebo.urdf.xacro" />
@@ -173,5 +184,6 @@
       <origin xyz="0.4288 0.2358 0.1914" rpy="0.0 0.0 ${0.25 * pi}" />  <!-- from visually matching up the meshes of the MiR and the laser scanner -->
     </joint>
-    <xacro:sick_s300 prefix="${prefix}" link="front_laser_link" topic="f_scan" />
+    <xacro:sick_s300 prefix="${prefix}" link="front_laser_link" topic="f_scan"
+                     prepend_prefix_to_laser_frame="$(arg prepend_prefix_to_laser_frame)" />
     <joint name="${prefix}base_link_to_back_laser_joint" type="fixed">
       <parent link="${prefix}base_link" />
@@ -179,5 +191,6 @@
       <origin xyz="-0.3548 -0.2352 0.1914" rpy="0.0 0.0 ${-0.75 * pi}" />  <!-- from visually matching up the meshes of the MiR and the laser scanner -->
     </joint>
-    <xacro:sick_s300 prefix="${prefix}" link="back_laser_link" topic="b_scan" />
+    <xacro:sick_s300 prefix="${prefix}" link="back_laser_link" topic="b_scan"
+                     prepend_prefix_to_laser_frame="$(arg prepend_prefix_to_laser_frame)" />
     <!-- Ultrasound sensors -->
     <joint name="${prefix}us_1_joint" type="fixed">   <!-- right ultrasound -->
@@ -210,5 +223,5 @@
     <!-- set the gazebo friction parameters for the wheels -->
     <xacro:set_all_wheel_frictions prefix="${prefix}"/>
-    <p3d_base_controller prefix="${prefix}" />
+    <xacro:p3d_base_controller prefix="${prefix}" />
   </xacro:macro>
 </robot>

File: mir_description/urdf/include/sick_s300.urdf.xacro (robot description, xacro)
@@ -6,5 +6,5 @@
   <xacro:property name="laser_z" value="0.185" />
   <xacro:property name="laser_mass" value="2.0" />
-  <xacro:macro name="sick_s300" params="link topic prefix">
+  <xacro:macro name="sick_s300" params="link topic prefix prepend_prefix_to_laser_frame='false'">
     <link name="${prefix}${link}">
       <visual>
@@ -57,6 +57,20 @@
         </ray>
         <plugin name="gazebo_ros_${link}_controller" filename="libgazebo_ros_laser.so">
-          <!-- no prefix, plugin always uses a tf_prefix (if none is set it uses robotNamespace) -->
-          <frameName>${link}</frameName>
+          <!-- The gazebo_ros_laser plugin does the following:
+               - If the ROS parameter 'tf_prefix' is set, it prepends the
+               - tf_prefix in front of the frameName.
+               - Otherwise, it prepends the robotNamespace.
+               The robotNamespace gets automatically set if you start the
+               spawn_model node inside a namespace. In this case, set
+               prepend_prefix_to_laser_frame to 'false', otherwise the
+               resulting frameName will have two prefixes prepended.
+               If you don't start spawn_model inside a namespace but have a
+               non-empty prefix, set prepend_prefix_to_laser_frame to 'true'. -->
+          <xacro:if value="${prepend_prefix_to_laser_frame}">
+            <frameName>${prefix}${link}</frameName>
+          </xacro:if>
+          <xacro:unless value="${prepend_prefix_to_laser_frame}">
+            <frameName>${link}</frameName>
+          </xacro:unless>
           <topicName>${topic}</topicName>
         </plugin>

File: mir_description/urdf/mir.urdf.xacro (robot description, xacro)
@@ -5,5 +5,13 @@
   <xacro:include filename="$(find mir_description)/urdf/include/mir_100_v1.urdf.xacro" />
   <xacro:include filename="$(find mir_description)/urdf/include/common.gazebo.xacro" />
-  <xacro:mir_100 prefix=""/>
+  <xacro:arg name="tf_prefix" default="" />
+  <xacro:property name="tf_prefix_" value="$(arg tf_prefix)" />
+  <xacro:if value="${tf_prefix_ == ''}">
+    <xacro:property name="prefix" value="" />
+  </xacro:if>
+  <xacro:unless value="${tf_prefix_ == ''}">
+    <xacro:property name="prefix" value="${tf_prefix_}/" />
+  </xacro:unless>
+  <xacro:mir_100 prefix="${prefix}"/>
   <xacro:controller_plugin_gazebo robot_namespace=""/>
   <!-- instead of the controller_plugin_gazebo, you can use the diffdrive controller like this:
