Commit message: Imported upstream version '1.1.2' of 'upstream'

File: mir_description/urdf/include/mir_100_v1.urdf.xacro (robot description, xacro)
@@ -1,15 +1,4 @@
 <?xml version="1.0"?>
 <robot xmlns:xacro="http://ros.org/wiki/xacro">
-  <!-- The gazebo_ros_laser plugin does the following:
-       - If the ROS parameter 'tf_prefix' is set, it prepends the
-       - tf_prefix in front of the frameName.
-       - Otherwise, it prepends the robotNamespace.
-       The robotNamespace gets automatically set if you start the
-       spawn_model node inside a namespace. In this case, set
-       prepend_prefix_to_laser_frame to 'false', otherwise the
-       resulting frameName will have two prefixes prepended.
-       If you don't start spawn_model inside a namespace but have a
-       non-empty prefix, set prepend_prefix_to_laser_frame to 'true'. -->
-  <xacro:arg name="prepend_prefix_to_laser_frame" default="false" />
   <xacro:include filename="$(find mir_description)/urdf/include/common_properties.urdf.xacro" />
   <xacro:include filename="$(find mir_description)/urdf/include/imu.gazebo.urdf.xacro" />
@@ -184,6 +173,5 @@
       <origin xyz="0.4288 0.2358 0.1914" rpy="0.0 0.0 ${0.25 * pi}" />  <!-- from visually matching up the meshes of the MiR and the laser scanner -->
     </joint>
-    <xacro:sick_s300 prefix="${prefix}" link="front_laser_link" topic="f_scan"
-                     prepend_prefix_to_laser_frame="$(arg prepend_prefix_to_laser_frame)" />
+    <xacro:sick_s300 prefix="${prefix}" link="front_laser_link" topic="f_scan" />
     <joint name="${prefix}base_link_to_back_laser_joint" type="fixed">
       <parent link="${prefix}base_link" />
@@ -191,6 +179,5 @@
       <origin xyz="-0.3548 -0.2352 0.1914" rpy="0.0 0.0 ${-0.75 * pi}" />  <!-- from visually matching up the meshes of the MiR and the laser scanner -->
     </joint>
-    <xacro:sick_s300 prefix="${prefix}" link="back_laser_link" topic="b_scan"
-                     prepend_prefix_to_laser_frame="$(arg prepend_prefix_to_laser_frame)" />
+    <xacro:sick_s300 prefix="${prefix}" link="back_laser_link" topic="b_scan" />
     <!-- Ultrasound sensors -->
     <joint name="${prefix}us_1_joint" type="fixed">   <!-- right ultrasound -->

File: mir_description/urdf/include/sick_s300.urdf.xacro (robot description, xacro)
@@ -6,5 +6,5 @@
   <xacro:property name="laser_z" value="0.185" />
   <xacro:property name="laser_mass" value="2.0" />
-  <xacro:macro name="sick_s300" params="link topic prefix prepend_prefix_to_laser_frame='false'">
+  <xacro:macro name="sick_s300" params="link topic prefix">
     <link name="${prefix}${link}">
       <visual>
@@ -57,20 +57,5 @@
         </ray>
         <plugin name="gazebo_ros_${link}_controller" filename="libgazebo_ros_laser.so">
-          <!-- The gazebo_ros_laser plugin does the following:
-               - If the ROS parameter 'tf_prefix' is set, it prepends the
-               - tf_prefix in front of the frameName.
-               - Otherwise, it prepends the robotNamespace.
-               The robotNamespace gets automatically set if you start the
-               spawn_model node inside a namespace. In this case, set
-               prepend_prefix_to_laser_frame to 'false', otherwise the
-               resulting frameName will have two prefixes prepended.
-               If you don't start spawn_model inside a namespace but have a
-               non-empty prefix, set prepend_prefix_to_laser_frame to 'true'. -->
-          <xacro:if value="${prepend_prefix_to_laser_frame}">
-            <frameName>${prefix}${link}</frameName>
-          </xacro:if>
-          <xacro:unless value="${prepend_prefix_to_laser_frame}">
-            <frameName>${link}</frameName>
-          </xacro:unless>
+          <frameName>${prefix}${link}</frameName>
           <topicName>${topic}</topicName>
         </plugin>

Commit message: Imported upstream version '1.0.8' of 'upstream'

File: mir_description/urdf/include/mir_100_v1.urdf.xacro (robot description, xacro)
@@ -1,4 +1,15 @@
 <?xml version="1.0"?>
 <robot xmlns:xacro="http://ros.org/wiki/xacro">
+  <!-- The gazebo_ros_laser plugin does the following:
+       - If the ROS parameter 'tf_prefix' is set, it prepends the
+       - tf_prefix in front of the frameName.
+       - Otherwise, it prepends the robotNamespace.
+       The robotNamespace gets automatically set if you start the
+       spawn_model node inside a namespace. In this case, set
+       prepend_prefix_to_laser_frame to 'false', otherwise the
+       resulting frameName will have two prefixes prepended.
+       If you don't start spawn_model inside a namespace but have a
+       non-empty prefix, set prepend_prefix_to_laser_frame to 'true'. -->
+  <xacro:arg name="prepend_prefix_to_laser_frame" default="false" />
   <xacro:include filename="$(find mir_description)/urdf/include/common_properties.urdf.xacro" />
   <xacro:include filename="$(find mir_description)/urdf/include/imu.gazebo.urdf.xacro" />
@@ -173,5 +184,6 @@
       <origin xyz="0.4288 0.2358 0.1914" rpy="0.0 0.0 ${0.25 * pi}" />  <!-- from visually matching up the meshes of the MiR and the laser scanner -->
     </joint>
-    <xacro:sick_s300 prefix="${prefix}" link="front_laser_link" topic="f_scan" />
+    <xacro:sick_s300 prefix="${prefix}" link="front_laser_link" topic="f_scan"
+                     prepend_prefix_to_laser_frame="$(arg prepend_prefix_to_laser_frame)" />
     <joint name="${prefix}base_link_to_back_laser_joint" type="fixed">
       <parent link="${prefix}base_link" />
@@ -179,5 +191,6 @@
       <origin xyz="-0.3548 -0.2352 0.1914" rpy="0.0 0.0 ${-0.75 * pi}" />  <!-- from visually matching up the meshes of the MiR and the laser scanner -->
     </joint>
-    <xacro:sick_s300 prefix="${prefix}" link="back_laser_link" topic="b_scan" />
+    <xacro:sick_s300 prefix="${prefix}" link="back_laser_link" topic="b_scan"
+                     prepend_prefix_to_laser_frame="$(arg prepend_prefix_to_laser_frame)" />
     <!-- Ultrasound sensors -->
     <joint name="${prefix}us_1_joint" type="fixed">   <!-- right ultrasound -->

File: mir_description/urdf/include/sick_s300.urdf.xacro (robot description, xacro)
@@ -6,5 +6,5 @@
   <xacro:property name="laser_z" value="0.185" />
   <xacro:property name="laser_mass" value="2.0" />
-  <xacro:macro name="sick_s300" params="link topic prefix">
+  <xacro:macro name="sick_s300" params="link topic prefix prepend_prefix_to_laser_frame='false'">
     <link name="${prefix}${link}">
       <visual>
@@ -57,5 +57,20 @@
         </ray>
         <plugin name="gazebo_ros_${link}_controller" filename="libgazebo_ros_laser.so">
-          <frameName>${prefix}${link}</frameName>
+          <!-- The gazebo_ros_laser plugin does the following:
+               - If the ROS parameter 'tf_prefix' is set, it prepends the
+               - tf_prefix in front of the frameName.
+               - Otherwise, it prepends the robotNamespace.
+               The robotNamespace gets automatically set if you start the
+               spawn_model node inside a namespace. In this case, set
+               prepend_prefix_to_laser_frame to 'false', otherwise the
+               resulting frameName will have two prefixes prepended.
+               If you don't start spawn_model inside a namespace but have a
+               non-empty prefix, set prepend_prefix_to_laser_frame to 'true'. -->
+          <xacro:if value="${prepend_prefix_to_laser_frame}">
+            <frameName>${prefix}${link}</frameName>
+          </xacro:if>
+          <xacro:unless value="${prepend_prefix_to_laser_frame}">
+            <frameName>${link}</frameName>
+          </xacro:unless>
           <topicName>${topic}</topicName>
         </plugin>
