Commit message: Imported upstream version '1.0.3' of 'upstream'

File: mir_description/urdf/include/imu.gazebo.urdf.xacro (robot description, xacro)
@@ -1,4 +1,13 @@
 <?xml version="1.0"?>
 <robot xmlns:xacro="http://ros.org/wiki/xacro">
+  <!-- If tf_prefix is given, use "frame tf_prefix/imu_frame", else "imu_frame" -->
+  <xacro:arg name="tf_prefix" default="" />
+  <xacro:property name="tf_prefix" value="$(arg tf_prefix)" />
+  <xacro:if value="${tf_prefix == ''}">
+      <xacro:property name="imu_frame" value="imu_frame" />
+  </xacro:if>
+  <xacro:unless value="${tf_prefix == ''}">
+      <xacro:property name="imu_frame" value="$(arg tf_prefix)/imu_frame" />
+  </xacro:unless>
   <xacro:macro name="imu_gazebo" params="link imu_topic update_rate stdev">
     <gazebo reference="${link}">
@@ -16,5 +25,5 @@
           <xyzOffset>0 0 0</xyzOffset>
           <rpyOffset>0 0 0</rpyOffset>
-          <frameName>imu_frame</frameName>  <!-- from real MiR -->
+          <frameName>${imu_frame}</frameName>  <!-- from real MiR -->
         </plugin>
         <pose>0 0 0 0 0 0</pose>

File: mir_description/urdf/include/mir_100_v1.urdf.xacro (robot description, xacro)
@@ -173,5 +173,5 @@
       <origin xyz="0.4288 0.2358 0.1914" rpy="0.0 0.0 ${0.25 * pi}" />  <!-- from visually matching up the meshes of the MiR and the laser scanner -->
     </joint>
-    <xacro:sick_s300 link="${prefix}front_laser_link" topic="f_scan" />
+    <xacro:sick_s300 prefix="${prefix}" link="front_laser_link" topic="f_scan" />
     <joint name="${prefix}base_link_to_back_laser_joint" type="fixed">
       <parent link="${prefix}base_link" />
@@ -179,5 +179,18 @@
       <origin xyz="-0.3548 -0.2352 0.1914" rpy="0.0 0.0 ${-0.75 * pi}" />  <!-- from visually matching up the meshes of the MiR and the laser scanner -->
     </joint>
-    <xacro:sick_s300 link="${prefix}back_laser_link" topic="b_scan" />
+    <xacro:sick_s300 prefix="${prefix}" link="back_laser_link" topic="b_scan" />
+    <!-- Ultrasound sensors -->
+    <joint name="${prefix}us_1_joint" type="fixed">   <!-- right ultrasound -->
+      <parent link="${prefix}base_link" />
+      <child link="${prefix}us_1_frame" />
+      <origin xyz="0.45 -0.12 0.16 " rpy="0 0 0" />  <!-- from visually matching to the mesh of the MiR -->
+    </joint>
+    <link name="${prefix}us_1_frame" />
+    <joint name="${prefix}us_2_joint" type="fixed">   <!-- left ultrasound -->
+      <parent link="${prefix}base_link" />
+      <child link="${prefix}us_2_frame" />
+      <origin xyz="0.45 0.12 0.16 " rpy="0 0 0" />  <!-- from visually matching to the mesh of the MiR -->
+    </joint>
+    <link name="${prefix}us_2_frame" />
     <!-- wheels -->
     <xacro:actuated_wheel prefix="${prefix}" locationprefix="left" locationright="-1"/>

File: mir_description/urdf/include/sick_s300.urdf.xacro (robot description, xacro)
@@ -6,6 +6,6 @@
   <xacro:property name="laser_z" value="0.185" />
   <xacro:property name="laser_mass" value="2.0" />
-  <xacro:macro name="sick_s300" params="link topic">
-    <link name="${link}">
+  <xacro:macro name="sick_s300" params="link topic prefix">
+    <link name="${prefix}${link}">
       <visual>
         <origin xyz="0.0 0.0 0.0" rpy="${pi} 0 0" />
@@ -26,8 +26,8 @@
       </xacro:box_inertial>
     </link>
-    <gazebo reference="${link}">
+    <gazebo reference="${prefix}${link}">
       <!-- <material value="Gazebo/Yellow" /> -->
       <material value="Gazebo/FlatBlack" />
-      <sensor type="gpu_ray" name="${link}">
+      <sensor type="gpu_ray" name="${prefix}${link}">
         <pose>0 0 0 0 0 0</pose>
         <visualize>false</visualize>
@@ -57,4 +57,5 @@
         </ray>
         <plugin name="gazebo_ros_${link}_controller" filename="libgazebo_ros_gpu_laser.so">
+          <!-- no prefix, plugin always uses a tf_prefix (if none is set it uses robotNamespace) -->
           <frameName>${link}</frameName>
           <topicName>${topic}</topicName>

Commit message: Imported upstream version '1.1.4' of 'upstream'

File: mir_description/urdf/include/imu.gazebo.urdf.xacro (robot description, xacro)
@@ -10,23 +10,19 @@
       <xacro:property name="imu_frame" value="$(arg tf_prefix)/imu_frame" />
   </xacro:unless>
-  <xacro:macro name="imu_gazebo" params="link imu_topic update_rate stdev">
-    <gazebo reference="${link}">
-      <gravity>true</gravity>
-      <sensor name="imu_sensor" type="imu">
-        <always_on>true</always_on>
-        <update_rate>100</update_rate>  <!-- this is not the publish rate -->
-        <visualize>true</visualize>
-        <topic>__default_topic__</topic>
-        <plugin filename="libgazebo_ros_imu_sensor.so" name="imu_plugin">
-          <topicName>${imu_topic}</topicName>
-          <bodyName>${link}</bodyName>
-          <updateRateHZ>${update_rate}</updateRateHZ>  <!-- this is the publish rate -->
-          <gaussianNoise>${stdev * stdev}</gaussianNoise>
-          <xyzOffset>0 0 0</xyzOffset>
-          <rpyOffset>0 0 0</rpyOffset>
-          <frameName>${imu_frame}</frameName>  <!-- from real MiR -->
-        </plugin>
-        <pose>0 0 0 0 0 0</pose>
-      </sensor>
+  <xacro:macro name="imu_gazebo" params="link imu_topic update_rate">
+    <gazebo>
+      <plugin name="imu_plugin" filename="libhector_gazebo_ros_imu.so">
+        <updateRate>${update_rate}</updateRate>
+        <!-- <robotNamespace>$(arg robot_namespace)</robotNamespace> -->
+        <bodyName>${link}</bodyName>
+        <frameId>${imu_frame}</frameId>  <!-- from real MiR -->
+        <topicName>${imu_topic}</topicName>
+        <accelDrift>0.0 0.0 0.0</accelDrift>
+        <accelGaussianNoise>${sqrt(5e-05)} ${sqrt(0.0001)} ${sqrt(0.00013)}</accelGaussianNoise>    <!-- real MiR linear_acceleration_covariance: [5e-05, 0.0, 0.0, 0.0, 0.0001, 0.0, 0.0, 0.0, 0.00013] -->
+        <rateDrift>0.0 0.0 0.0</rateDrift>
+        <rateGaussianNoise>${sqrt(8e-06)} ${sqrt(8e-06)} ${sqrt(3e-07)}</rateGaussianNoise>         <!-- real MiR angular_velocity_covariance: [8e-06, 0.0, 0.0, 0.0, 8e-06, 0.0, 0.0, 0.0, 3e-07] -->
+        <yawDrift>0.0</yawDrift>
+        <yawGaussianNoise>${sqrt(0.1)}</yawGaussianNoise>                                           <!-- real MiR orientation_covariance: [0.1, 0.0, 0.0, 0.0, 0.1, 0.0, 0.0, 0.0, 0.1] -->
+      </plugin>
     </gazebo>
   </xacro:macro>

File: mir_description/urdf/include/mir_100_v1.urdf.xacro (robot description, xacro)
@@ -23,5 +23,4 @@
   <xacro:property name="mir_100_caster_wheel_base_dy" value="0.203" />
   <xacro:property name="mir_100_caster_wheel_base_dz" value="${mir_100_caster_wheel_radius-mir_100_caster_wheel_dz}" />
-  <xacro:property name="imu_stdev" value="0.00017" />
   <xacro:macro name="actuated_wheel" params="prefix locationprefix locationright">
     <joint name="${prefix}${locationprefix}_wheel_joint" type="continuous">
@@ -44,7 +43,7 @@
       </visual>
       <collision>
-        <origin xyz="0 0 0" rpy="0 0 0" />
-        <geometry>
-          <mesh filename="package://mir_description/meshes/visual/wheel.stl" />
+        <origin xyz="0 0 0" rpy="${pi/2} 0 0" />
+        <geometry>
+          <cylinder radius="${mir_100_act_wheel_radius}" length="${mir_100_act_wheel_width}" />
         </geometry>
       </collision>
@@ -112,7 +111,7 @@
       </visual>
       <collision>
-        <origin xyz="0 0 0" rpy="0 0 0" />
-        <geometry>
-          <mesh filename="package://mir_description/meshes/visual/wheel.stl" />
+        <origin xyz="0 0 0" rpy="${pi/2} 0 0" />
+        <geometry>
+          <cylinder radius="${mir_100_caster_wheel_radius}" length="${mir_100_caster_wheel_width}" />
         </geometry>
       </collision>
@@ -157,5 +156,5 @@
     </joint>
     <link name="${prefix}imu_link" />
-    <xacro:imu_gazebo link="${prefix}imu_link" imu_topic="imu_data" update_rate="50.0" stdev="${imu_stdev}" />
+    <xacro:imu_gazebo link="${prefix}imu_link" imu_topic="imu_data" update_rate="50.0" />
     <!-- Create an alias for imu_link. This is necessary because the real MiR's
          TF has imu_link, but the imu_data topic is published in the imu_frame
